Commit message: fix robot bug

File: src/vica_robot/urdf/macros.xacro (robot description, xacro)
@@ -1,70 +1,3 @@
 <?xml version="1.0"?>
 <robot>
-  <!--
-  macro name="cylinder_inertia" params="m r h">
-    <inertia  ixx="${m*(3*r*r+h*h)/12}" ixy = "0" ixz = "0"
-      iyy="${m*(3*r*r+h*h)/12}" iyz = "0"
-      izz="${m*r*r/2}"
-    />
-  </macro>
-  <macro name="box_inertia" params="m x y z">
-    <inertia  ixx="${m*(y*y+z*z)/12}" ixy = "0" ixz = "0"
-      iyy="${m*(x*x+z*z)/12}" iyz = "0"
-      izz="${m*(x*x+z*z)/12}"
-    />
-  </macro>
-  <macro name="sphere_inertia" params="m r">
-    <inertia  ixx="${2*m*r*r/5}" ixy = "0" ixz = "0"
-      iyy="${2*m*r*r/5}" iyz = "0"
-      izz="${2*m*r*r/5}"
-    />
-  </macro>
-  <macro name="wheel" params="lr tY">
-    <link name="${lr}_wheel">
-      <collision>
-        <origin xyz="0 0 0" rpy="0 ${PI/2} ${PI/2}" />
-        <geometry>
-          <cylinder length="${wheelWidth}" radius="${wheelRadius}"/>
-        </geometry>
-      </collision>
-      <visual>
-        <origin xyz="0 0 0" rpy="0 ${PI/2} ${PI/2}" />
-        <geometry>
-          <cylinder length="${wheelWidth}" radius="${wheelRadius}"/>
-        </geometry>
-        <material name="black"/>
-      </visual>
-      <inertial>
-        <origin xyz="0 0 0" rpy="0 ${PI/2} ${PI/2}" />
-        <mass value="${wheelMass}"/>
-        <cylinder_inertia m="${wheelMass}" r="${wheelRadius}" h="${wheelWidth}"/>
-      </inertial>
-    </link>
-    <gazebo reference="${lr}_wheel">
-      <mu1 value="1.0"/>
-      <mu2 value="1.0"/>
-      <kp  value="10000000.0" />
-      <kd  value="1.0" />
-      <fdir1 value="1 0 0"/>
-      <material>Gazebo/Black</material>
-    </gazebo>
-    <joint name="${lr}_wheel_hinge" type="continuous">
-      <parent link="chassis"/>
-      <child link="${lr}_wheel"/>
-    <origin xyz="${-wheelPos+chassisLength/2} ${tY*wheelWidth/2+tY*chassisWidth/2} ${wheelRadius}" rpy="0 0 0" />
-      <axis xyz="0 1 0" rpy="0 0 0" />
-      <limit effort="10000" velocity="10000"/>
-      <joint_properties damping="0.0" friction="0.0"/>
-    </joint>
-    <transmission name="${lr}_trans">
-      <type>transmission_interface/SimpleTransmission</type>
-      <joint name="${lr}_wheel_hinge">
-        <hardwareInterface>EffortJointInterface</hardwareInterface>
-      </joint>
-      <actuator name="${lr}Motor">
-        <hardwareInterface>EffortJointInterface</hardwareInterface>
-        <mechanicalReduction>10</mechanicalReduction>
-      </actuator>
-    </transmission>
-  </macro-->
 </robot>

File: src/vica_robot/urdf/model_tmp2.xacro (robot description, xacro)
@@ -1,10 +1,7 @@
 <?xml version="1.0"?>
 <robot name="ubot" xmlns:xacro="http://www.ros.org/wiki/xacro">
-	<xacro:include
-		filename="$(find vica_robot)/urdf/robot.gazebo" />
-	<xacro:include
-		filename="$(find vica_robot)/urdf/materials.xacro" />
-	<xacro:include
-		filename="$(find vica_robot)/urdf/macros.xacro" />
+	<xacro:include filename="$(find vica_robot)/urdf/robot.gazebo" />
+	<xacro:include filename="$(find vica_robot)/urdf/materials.xacro" />
+	<xacro:include filename="$(find vica_robot)/urdf/macros.xacro" />
 	<robotBaseFrame>base_link</robotBaseFrame>
 	<link name="base_link">
@@ -12,6 +9,5 @@
 			<origin rpy="0 0 0" xyz="0 0 0.05" />
 			<geometry>
-				<mesh scale=".0010 .0010 .0010"
-					filename="package://vica_robot/meshes/base.stl" />
+				<mesh scale=".0010 .0010 .0010" filename="package://vica_robot/meshes/base.stl" />
 			</geometry>
 			<material name="Yellow">
@@ -22,11 +18,10 @@
 			<origin rpy="0 0 0" xyz="0 0 0.05" />
 			<geometry>
-				<mesh scale=".0010 .0010 .0010"
-					filename="package://vica_robot/meshes/base.stl" />
-			</geometry>
-		</collision>
-		<inertial>
-			<mass value="5" />
-			<origin xyz="0 0 0" rpy="0 0 0" />
+				<mesh scale=".0010 .0010 .0010" filename="package://vica_robot/meshes/base.stl" />
+			</geometry>
+		</collision>
+		<inertial>
+			<origin rpy="0 0 0" xyz="0 0 0" />
+			<mass value="5.0" />
 			<inertia ixx="0.88" ixy="0" ixz="0"
 					 iyy="0.88" iyz="0"
@@ -37,104 +32,78 @@
 	<link name="caster_front_link">
 		<visual>
-			<origin xyz="0.135 0 0.0325" rpy="0 0 0" />
-			<geometry>
-				<sphere radius="0.03" />
+			<origin xyz="0 0 0.0051" rpy="0 0 0" />
+			<geometry>
+				<sphere radius="0.005" />
 			</geometry>
 		</visual>
 		<collision name='caster_front_collision'>
-			<origin xyz="0.135 0 0.0325" rpy="0 0 0" />
-			<geometry>
-				<sphere radius="0.03" />
-			</geometry>
-			<surface>
-				<friction>
-					<ode>
-						<mu>0.01</mu>
-						<mu2>0.01</mu2>
-						<fdir1> 0 0 0</fdir1>
-						<slip1>1.0</slip1>
-						<slip2>1.0</slip2>
-					</ode>
-				</friction>
-				<bounce>
-					<restitution_coefficient>0</restitution_coefficient>
-					<threshold>100000</threshold>
-				</bounce>
-				<contact>
-					<ode>
-						<soft_cfm>0</soft_cfm>
-						<soft_erp>0.2</soft_erp>
-						<kp>1.0</kp>
-						<kd>1.0</kd>
-						<max_vel>1.0</max_vel>
-						<min_depth>0.001</min_depth>
-					</ode>
-				</contact>
-			</surface>
-		</collision>
-		<inertial>
-			<mass value="0.01" />
-			<inertia ixx="0.001" ixy="0.0" ixz="0.0"
-                     iyy="0.001" iyz="0.0"
-					 izz="0.001" />
+			<origin xyz="0 0.00 0.0051" rpy="0 0 0" />
+			<geometry>
+				<sphere radius="0.005" />
+			</geometry>
+			<surface>
+				 <friction>
+            		<ode>
+		                <mu>00.000000</mu>
+		                <mu2>00.000000</mu2>
+		                <slip1>1.0</slip1>
+		                <slip2>1.0</slip2>
+              		</ode>
+            	</friction>
+			</surface>
+		</collision>
+		<inertial>
+        	<mass value="0.01" />
+        	<origin xyz="0 0.00 0.005" rpy="0 0 0.005" />
+        	<inertia ixx="0.001" ixy="0.0" ixz="0.0"
+                	 iyy="0.001" iyz="0.0"
+                 	izz="0.001" />
 		</inertial>
 	</link>
 	<joint name="caster_front_join" type="fixed">
-		<parent link="base_link" />
-		<child link="caster_front_link" />
-		<origin xyz="0 0 0.0001" rpy="0 0 0" />
+	      <parent link="base_link"/>
+	      <child link="caster_front_link"/>
+	      <origin xyz="0.135 0 0.005" rpy="0 0 0" />
 	</joint>
 	<!-- Fin Roue libre devant -->
-	<!-- Roue libre arriere -->
+	<!-- Roue libre arriere
 	<link name="caster_back_link">
 		<visual>
-			<origin xyz="-0.135 0 0.0325" rpy="0 0 0" />
-			<geometry>
-				<sphere radius="0.03" />
+			<origin xyz="0.135 0.00 0.005" rpy="0 0 0" />
+			<geometry>
+				<sphere radius="0.005" />
 			</geometry>
 		</visual>
 		<collision name='caster_back_collision'>
-			<origin xyz="-0.135 0 0.0325" rpy="0 0 0" />
-			<geometry>
-				<sphere radius="0.03" />
-			</geometry>
-			<surface>
-				<friction>
-					<ode>
-						<mu>0.01</mu>
-						<mu2>0.01</mu2>
-						<fdir1> 0 0 0</fdir1>
-						<slip1>1.0</slip1>
-						<slip2>1.0</slip2>
-					</ode>
-				</friction>
-				<bounce>
-					<restitution_coefficient>0</restitution_coefficient>
-					<threshold>100000</threshold>
-				</bounce>
-				<contact>
-					<ode>
-						<soft_cfm>0</soft_cfm>
-						<soft_erp>0.2</soft_erp>
-						<kp>1.0</kp>
-						<kd>1.0</kd>
-						<max_vel>1.0</max_vel>
-						<min_depth>0.001</min_depth>
-					</ode>
-				</contact>
-			</surface>
-		</collision>
-		<inertial>
-			<mass value="0.01"/>
-			<inertia ixx="0.001" ixy="0.0" ixz="0.0"
-               		   iyy="0.001" iyz="0.0"
-					   izz="0.001" />
+			<origin xyz="0.135 0.00 0.005" rpy="0 0 0" />
+			<geometry>
+				<sphere radius="0.005" />
+			</geometry>
+			<surface>
+				 <friction>
+            		<ode>
+		                <mu>00.000000</mu>
+		                <mu2>00.000000</mu2>
+		                <fdir1>0.000000 0.000000 0.000000</fdir1>
+		                <slip1>0.000000</slip1>
+		                <slip2>0.000000</slip2>
+              		</ode>
+                 </friction>
+			</surface>
+		</collision>
+		<inertial>
+        	<mass value="0.01" />
+        	<origin xyz="0.135 0.00 0.005" rpy="0 0 0" />
+        	<inertia ixx="0.001" ixy="0.0" ixz="0.0"
+                    iyy="0.001" iyz="0.0"
+                     izz="0.001" />
 		</inertial>
 	</link>
 	<joint name="caster_back_join" type="fixed">
-		<parent link="base_link" />
-		<child link="caster_back_link" />
-		<origin xyz="0 0 0.0001" rpy="0 0 0" />
-	</joint>
+	      <parent link="base_link"/>
+	      <child link="caster_back_link"/>
+	      <origin xyz="0 0 0.005" rpy="0 0 0" />
+	</joint>
+		-->
 	<!-- Fin Roue libre arriere -->
 	<link name="r_wheel">
@@ -142,7 +111,6 @@
 			<origin rpy="0 1.57079632679 0" xyz="0 0 0" />
 			<geometry>
-				<!-- <mesh scale=".0010 .0010 .0010" filename="package://vica_robot/meshes/rwheel.stl"
-					/> -->
-				<cylinder length="0.025" radius="0.03" />
+				<!--   <mesh scale=".0010 .0010 .0010" filename="package://vica_robot/meshes/rwheel.stl" />-->
+				<cylinder length="0.025" radius="0.03"/>
 			</geometry>
 			<material name="Blue">
@@ -153,7 +121,6 @@
 			<origin rpy="0 1.57079632679 0" xyz="0 0 0" />
 			<geometry>
-				<!-- <mesh scale=".0010 .0010 .0010" filename="package://vica_robot/meshes/rwheel.stl"
-					/> -->
-				<cylinder length="0.025" radius="0.03" />
+				<!--   <mesh scale=".0010 .0010 .0010" filename="package://vica_robot/meshes/rwheel.stl" />-->
+				<cylinder length="0.025" radius="0.03"/>
 			</geometry>
 			<surface>
@@ -163,18 +130,17 @@
 						<mu2>1.0</mu2>
 						<slip1>0.0</slip1>
-						<slip2>0.0</slip2>
+          				<slip2>0.0</slip2>
 					</ode>
 				</friction>
 				<contact>
-					<ode>
-					</ode>
-				</contact>
-			</surface>
-		</collision>
-		<inertial>
-			<mass value="5" />
+              	   <ode>
+	               </ode>
+	            </contact>
+			</surface>
+		</collision>
+		<inertial>
+			<mass value="0.300" />
 			<cylinder_inertia m="5" r="0.1" h="0.05" />
-			<inertia ixx="0.89" ixy="0" ixz="0" iyy="1.0" iyz="0"
-				izz="0.88" />
+			<inertia ixx="0.89" ixy="0" ixz="0" iyy="1.0" iyz="0" izz="0.88" />
 		</inertial>
 	</link>
@@ -182,5 +148,5 @@
 		<parent link="base_link" />
 		<child link="r_wheel" />
-		<origin xyz="0 -0.15 0.0325" rpy="0 0 1.57079632679" />
+		<origin xyz="-0.14 -0.135 0.0325" rpy="0 0 1.57079632679" />
 	</joint>
 	<transmission name="r_wheel_transmission">
@@ -198,5 +164,5 @@
 			<origin rpy="0 1.57079632679 0" xyz="0 0 0" />
 			<geometry>
-				<cylinder length="0.025" radius="0.03" />
+				<cylinder length="0.025" radius="0.03"/>
 			</geometry>
 			<material name="Blue">
@@ -207,5 +173,5 @@
 			<origin rpy="0 1.57079632679 0" xyz="0 0 0" />
 			<geometry>
-				<cylinder length="0.025" radius="0.03" />
+				<cylinder length="0.025" radius="0.03"/>
 			</geometry>
 			<surface>
@@ -215,11 +181,11 @@
 						<mu2>1.0</mu2>
 						<slip1>0</slip1>
-						<slip2>0</slip2>
+          				<slip2>0</slip2>
 					</ode>
 				</friction>
 				<contact>
-					<ode>
-					</ode>
-				</contact>
+              	   <ode>
+	               </ode>
+	            </contact>
 			</surface>
 		</collision>
@@ -227,6 +193,5 @@
 			<mass value="0.300" />
 			<cylinder_inertia m="5" r="0.1" h="0.05" />
-			<inertia ixx="0.88" ixy="0" ixz="0" iyy="1.0" iyz="0"
-				izz="0.88" />
+			<inertia ixx="0.88" ixy="0" ixz="0" iyy="1.0" iyz="0" izz="0.88" />
 		</inertial>
 	</link>
@@ -234,5 +199,5 @@
 		<parent link="base_link" />
 		<child link="l_wheel" />
-		<origin xyz="0 0.15 0.0325" rpy="0 0 1.57079632679" />
+		<origin xyz="-0.14 0.135 0.0325" rpy="0 0 1.57079632679" />
 	</joint>
 	<transmission name="l_wheel_transmission">
@@ -250,6 +215,5 @@
 			<origin rpy="0 0 0" xyz="0 0 0" />
 			<geometry>
-				<mesh scale=".0010 .0010 .0010"
-					filename="package://vica_robot/meshes/kinect.stl" />
+				<mesh scale=".0010 .0010 .0010" filename="package://vica_robot/meshes/kinect.stl" />
 			</geometry>
 			<material name="Red">
@@ -259,12 +223,10 @@
 		<collision>
 			<geometry>
-				<mesh scale=".0010 .0010 .0010"
-					filename="package://vica_robot/meshes/kinect.stl" />
+				<mesh scale=".0010 .0010 .0010" filename="package://vica_robot/meshes/kinect.stl" />
 			</geometry>
 		</collision>
 		<inertial>
 			<mass value="0.681" />
-			<inertia ixx="0.89" ixy="0" ixz="0" iyy="1.0" iyz="0"
-				izz="0.89" />
+			<inertia ixx="0.89" ixy="0" ixz="0" iyy="1.0" iyz="0" izz="0.89" />
 		</inertial>
 	</link>
@@ -273,6 +235,5 @@
 			<origin rpy="1.57079632679 0 0" xyz="0 0 -0.04" />
 			<geometry>
-				<mesh scale=".0010 .0010 .0010"
-					filename="package://vica_robot/meshes/rplidar.stl" />
+				<mesh scale=".0010 .0010 .0010" filename="package://vica_robot/meshes/rplidar.stl" />
 			</geometry>
 			<material name="Red">
@@ -282,12 +243,10 @@
 		<collision>
 			<geometry>
-				<mesh scale=".0010 .0010 .0010"
-					filename="package://vica_robot/meshes/rplidar.stl" />
+				<mesh scale=".0010 .0010 .0010" filename="package://vica_robot/meshes/rplidar.stl" />
 			</geometry>
 		</collision>
 		<inertial>
 			<mass value="0.681" />
-			<inertia ixx="0.89" ixy="0" ixz="0" iyy="1.0" iyz="0"
-				izz="0.89" />
+			<inertia ixx="0.89" ixy="0" ixz="0" iyy="1.0" iyz="0" izz="0.89" />
 		</inertial>
 	</link>

File: src/vica_robot/urdf/model_tmp3_fonc.xacro (robot description, xacro)
@@ -135,5 +135,5 @@
 		<parent link="base_link" />
 		<child link="caster_back_link" />
-		<origin xyz="0 0 0.0001" rpy="0 0 0" />
+		<origin xyz="0 0 0.00010.0001" rpy="0 0 0" />
 	</joint>
 	<!-- Fin Roue libre arriere -->
