Commit message: fix bug LIDAR

File: src/vica_robot/urdf/model.xacro (robot description, xacro)
@@ -71,5 +71,5 @@
 	<link name="r_wheel">
 		<visual>
-			<origin rpy="0 0 1.58" xyz="0 0 0" />
+			<origin rpy="0 0 1.57079632679" xyz="0 0 0" />
 			<geometry>
 				<mesh scale=".0010 .0010 .0010" filename="package://vica_robot/meshes/rwheel.stl" />
@@ -80,5 +80,5 @@
 		</visual>
 		<collision>
-			<origin rpy="0 0 1.58" xyz="0 0 0" />
+			<origin rpy="0 0 1.57079632679" xyz="0 0 0" />
 			<geometry>
 				<mesh scale=".0010 .0010 .0010" filename="package://vica_robot/meshes/rwheel.stl" />
@@ -103,5 +103,5 @@
 	<link name="l_wheel">
 		<visual>
-			<origin rpy="0 0 1.58" xyz="0 0 0" />
+			<origin rpy="0 0 1.57079632679" xyz="0 0 0" />
 			<geometry>
 				<mesh scale=".0010 .0010 .0010" filename="package://vica_robot/meshes/lwheel.stl" />
@@ -112,5 +112,5 @@
 		</visual>
 		<collision>
-			<origin rpy="0 0 1.58" xyz="0 0 0" />
+			<origin rpy="0 0 1.57079632679" xyz="0 0 0" />
 			<geometry>
 				<mesh scale=".0010 .0010 .0010" filename="package://vica_robot/meshes/lwheel.stl" />
@@ -155,5 +155,5 @@
 	<link name="rplidar">
 		<visual>
-			<origin rpy="0 0 0" xyz="0 0 0" />
+			<origin rpy="1.57079632679 0 0" xyz="0 0 -0.04" />
 			<geometry>
 				<mesh scale=".0010 .0010 .0010" filename="package://vica_robot/meshes/rplidar.stl" />
@@ -176,10 +176,10 @@
 		<parent link="base_link" />
 		<child link="r_wheel" />
-		<origin xyz="0 -0.15 0.0325" rpy="0 0 1.58" />
+		<origin xyz="0 -0.15 0.0325" rpy="0 0 1.57079632679" />
 	</joint>
 	<joint name="l_wheel_joint" type="continuous">
 		<parent link="base_link" />
 		<child link="l_wheel" />
-		<origin xyz="0 0.15 0.0325" rpy="0 0 1.58" />
+		<origin xyz="0 0.15 0.0325" rpy="0 0 1.57079632679" />
 	</joint>
 	<joint name="kinect_joint" type="fixed">
@@ -191,5 +191,5 @@
 		<parent link="base_link" />
 		<child link="rplidar" />
-		<origin xyz="-0.06 0.033 0.238" rpy="1.58 0 0" />
+		<origin xyz="-0.06 0.033 0.28" rpy="0 0 0" />
 	</joint>
 </robot>

Commit message: fix robot

File: src/vica_robot/urdf/model.xacro (robot description, xacro)
@@ -27,5 +27,5 @@
 			<origin xyz="-0.135 0 0.01" rpy=" 0 0 0" />
 			<geometry>
-				<sphere radius="0.01" />
+				<sphere radius="0.012" />
 			</geometry>
 		</visual>
@@ -33,13 +33,13 @@
 			<origin xyz="-0.135 0 0.0325" rpy=" 0 0 0" />
 			<geometry>
-				<sphere radius="0.03245" />
-			</geometry>
-			<surface>
-				<friction>
-					<ode>
-						<mu>0</mu>
-						<mu2>0</mu2>
-						<slip1>1.0</slip1>
-						<slip2>1.0</slip2>
+				<sphere radius="0.012" />
+			</geometry>
+			<surface>
+				<friction>
+					<ode>
+		                  <mu>0</mu>
+		                  <mu2>0</mu2>
+		                  <slip1>1.0</slip1>
+		                  <slip2>1.0</slip2>
 					</ode>
 				</friction>
@@ -49,5 +49,5 @@
 			<origin xyz="0.135 0 0.01" rpy=" 0 0 0" />
 			<geometry>
-				<sphere radius="0.01" />
+				<sphere radius="0.012" />
 			</geometry>
 		</visual>
@@ -55,13 +55,13 @@
 			<origin xyz="0.135 0 0.0325" rpy=" 0 0 0" />
 			<geometry>
-				<sphere radius="0.03245" />
-			</geometry>
-			<surface>
-				<friction>
-					<ode>
-						<mu>0</mu>
-						<mu2>0</mu2>
-						<slip1>1.0</slip1>
-						<slip2>1.0</slip2>
+				<sphere radius="0.012" />
+			</geometry>
+			<surface>
+				<friction>
+					<ode>
+		                  <mu>0</mu>
+		                  <mu2>0</mu2>
+		                  <slip1>1.0</slip1>
+		                  <slip2>1.0</slip2>
 					</ode>
 				</friction>
@@ -87,8 +87,6 @@
 				<friction>
 					<ode>
-						<mu>1000000</mu>
+						<mu>100</mu>
 						<mu2>100</mu2>
-						<slip1>0</slip1>
-						<slip2>0</slip2>
 					</ode>
 				</friction>
@@ -98,5 +96,5 @@
 			<mass value="0.181" />
 			<cylinder_inertia m="5" r="0.1" h="0.05" />
-			<inertia ixx="0.89" ixy="0" ixz="0" iyy="1.0" iyz="0" izz="0.89" />
+			<inertia ixx="0.89" ixy="0" ixz="0" iyy="1.0" iyz="0" izz="0.88" />
 		</inertial>
 	</link>
@@ -119,8 +117,6 @@
 				<friction>
 					<ode>
-						<mu>1000000</mu>
+						<mu>100</mu>
 						<mu2>100</mu2>
-						<slip1>0</slip1>
-						<slip2>0</slip2>
 					</ode>
 				</friction>
@@ -178,4 +174,14 @@
 		<origin xyz="0 -0.15 0.0325" rpy="0 0 1.57079632679" />
 	</joint>
+	<transmission name="r_wheel_transmission">
+		<type>transmission_interface/SimpleTransmission</type>
+		<joint name="r_wheel_joint">
+			<hardwareInterface>hardware_interface/VelocityJointInterface</hardwareInterface>
+		</joint>
+		<actuator name="r_wheel_actuator">
+			<mechanicalReduction>7</mechanicalReduction>
+			<hardwareInterface>VelocityJointInterface</hardwareInterface>
+		</actuator>
+	</transmission>
 	<joint name="l_wheel_joint" type="continuous">
 		<parent link="base_link" />
@@ -183,4 +189,14 @@
 		<origin xyz="0 0.15 0.0325" rpy="0 0 1.57079632679" />
 	</joint>
+	<transmission name="l_wheel_transmission">
+		<type>transmission_interface/SimpleTransmission</type>
+		<joint name="l_wheel_joint">
+			<hardwareInterface>hardware_interface/VelocityJointInterface</hardwareInterface>
+		</joint>
+		<actuator name="l_wheel_actuator">
+			<mechanicalReduction>7</mechanicalReduction>
+			<hardwareInterface>VelocityJointInterface</hardwareInterface>
+		</actuator>
+	</transmission>
 	<joint name="kinect_joint" type="fixed">
 		<parent link="base_link" />

Commit message: fix bug move

File: src/vica_robot/urdf/model.xacro (robot description, xacro)
@@ -21,17 +21,17 @@
 		</collision>
 		<inertial>
-			<mass value="5.76" />
+			<mass value="20.76" />
 			<inertia ixx="0.88" ixy="0" ixz="0" iyy="1.0" iyz="0" izz="0.88" />
 		</inertial>
 		<visual name='caster_visual_front'>
-			<origin xyz="-0.135 0 0.01" rpy=" 0 0 0" />
-			<geometry>
-				<sphere radius="0.012" />
+			<origin xyz="-0.135 0.00 0.0035" rpy="0 0 0" />
+			<geometry>
+				<sphere radius="0.00339" />
 			</geometry>
 		</visual>
 		<collision name='caster_collision_front'>
-			<origin xyz="-0.135 0 0.0325" rpy=" 0 0 0" />
-			<geometry>
-				<sphere radius="0.012" />
+			<origin xyz="-0.135 0.00 0.0035" rpy="0 0 0" />
+			<geometry>
+				<sphere radius="0.00339" />
 			</geometry>
 			<surface>
@@ -47,13 +47,13 @@
 		</collision>
 		<visual name='caster_visual_back'>
-			<origin xyz="0.135 0 0.01" rpy=" 0 0 0" />
-			<geometry>
-				<sphere radius="0.012" />
+			<origin xyz="0.135 0.00 0.0035" rpy="0 0 0" />
+			<geometry>
+				<sphere radius="0.00339" />
 			</geometry>
 		</visual>
 		<collision name='caster_collision_back'>
-			<origin xyz="0.135 0 0.0325" rpy=" 0 0 0" />
-			<geometry>
-				<sphere radius="0.012" />
+			<origin xyz="0.135 0.00 0.0035" rpy="0 0 0" />
+			<geometry>
+				<sphere radius="0.00339" />
 			</geometry>
 			<surface>
@@ -87,6 +87,6 @@
 				<friction>
 					<ode>
-						<mu>100</mu>
-						<mu2>100</mu2>
+						<mu>1</mu>
+						<mu2>1</mu2>
 					</ode>
 				</friction>
@@ -117,6 +117,6 @@
 				<friction>
 					<ode>
-						<mu>100</mu>
-						<mu2>100</mu2>
+						<mu>1</mu>
+						<mu2>1</mu2>
 					</ode>
 				</friction>

Commit message: add graph topics

File: src/vica_robot/urdf/model.xacro (robot description, xacro)
@@ -10,5 +10,5 @@
 	<link name="base_link">
 		<visual>
-			<origin rpy="0 0 0" xyz="0 0 0.05" />
+			<origin rpy="0 0 0" xyz="0 0 0.01" />
 			<geometry>
 				<mesh scale=".0010 .0010 .0010"
@@ -20,5 +20,5 @@
 		</visual>
 		<collision>
-			<origin rpy="0 0 0" xyz="0 0 0.05" />
+			<origin rpy="0 0 0" xyz="0 0 0.01" />
 			<geometry>
 				<mesh scale=".0010 .0010 .0010"
